Commit message: test: complete Week 7 MuJoCo hardware acceptance

File: ros2_ws/src/robustlearn_description/urdf/panda.ros2_control.xacro (robot description, xacro)
@@ -1,8 +1,13 @@
 <?xml version="1.0"?>
 <robot xmlns:xacro="http://www.ros.org/wiki/xacro">
-  <xacro:macro name="panda_ros2_control" params="name">
+  <xacro:macro
+    name="panda_ros2_control"
+    params="name hardware_plugin model_path">
     <ros2_control name="${name}" type="system">
       <hardware>
-        <plugin>mock_components/GenericSystem</plugin>
+        <plugin>${hardware_plugin}</plugin>
+        <xacro:if value="${model_path != ''}">
+          <param name="model_path">${model_path}</param>
+        </xacro:if>
       </hardware>
       <joint name="panda_joint1">

File: ros2_ws/src/robustlearn_description/urdf/panda.urdf.xacro (robot description, xacro)
@@ -5,4 +5,10 @@
   <!-- ros2_control definition -->
   <xacro:include filename="panda.ros2_control.xacro"/>
+  <xacro:arg
+    name="hardware_plugin"
+    default="mock_components/GenericSystem"/>
+  <xacro:arg
+    name="model_path"
+    default=""/>
   <!-- Base -->
   <link name="panda_link0"/>
@@ -92,4 +98,7 @@
   </joint>
   <!-- Attach ros2_control hardware to the seven joints above -->
-  <xacro:panda_ros2_control name="PandaSystem"/>
+  <xacro:panda_ros2_control
+    name="PandaSystem"
+    hardware_plugin="$(arg hardware_plugin)"
+    model_path="$(arg model_path)"/>
 </robot>
